Commit message: fixed the issue with collisions

File: metal_head_v1m1_m4_with_arm_fixed_4/urdf/metal_head_v1m1_m4_with_arm_fixed_4.urdf (robot description, URDF)
Before this commit: robot metal_head, 19 links, 18 joints
Links:
- removed link Arm_Link
- added link base_inertia, mass 1.49829855979102
- link Link04_BL: geometry collision sphere radius=0.018; visual mesh filename=package://metal_head_v1m1_m4_with_arm_fixed_4/meshes/Link04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
- link Link04_BR: geometry collision sphere radius=0.018; visual mesh filename=package://metal_head_v1m1_m4_with_arm_fixed_4/meshes/Link04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
- link Link04_FL: geometry collision sphere radius=0.018; visual mesh filename=package://metal_head_v1m1_m4_with_arm_fixed_4/meshes/Link04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
- link Link04_FR: geometry collision sphere radius=0.018; visual mesh filename=package://metal_head_v1m1_m4_with_arm_fixed_4/meshes/Link04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
- link base: mass 1.49829855979102 -> None
Joints:
- removed joint Joint_01_arm
- added joint base_to_base_inertia: type fixed, parent base, child base_inertia, origin xyz=0 0 0 rpy=0 0 0
